File: Avionics/Avionics.kicad_pcb (KiCad board)
At the start: 2 copper layers, 91.1 x 91.1 mm, 9 parts, among them J1 Conn_02x03_Odd_Even, SW1 SW_SPST, U1 ATmega328P-A, Y1 Crystal_GND24

Commit message: 3hr
very tired
Parts:
- added C5: 100 nF, Capacitor_SMD:C_0805_2012Metric_Pad1.18x1.45mm_HandSolder, F.Cu at (145.0, 125.8)
- added C6: 100 nF, Capacitor_SMD:C_0805_2012Metric_Pad1.18x1.45mm_HandSolder, F.Cu at (145.0, 128.8)
- added C7: C, Capacitor_SMD:C_0805_2012Metric_Pad1.18x1.45mm_HandSolder, F.Cu at (145.0, 131.8)
- added C8: 1 uF, Capacitor_SMD:C_0805_2012Metric_Pad1.18x1.45mm_HandSolder, F.Cu at (128.5, 140.0)
- added C9: 0.1 uF, Capacitor_SMD:C_0805_2012Metric_Pad1.18x1.45mm_HandSolder, F.Cu at (134.5, 140.0)
- added D1: NeoPixel_THT, LED_SMD:LED_WS2812_PLCC6_5.0x5.0mm_P1.6mm, F.Cu at (138.5, 64.0)
- added D10: D, Diode_SMD:D_0201_0603Metric, F.Cu at (153.6, 126.9)
- added D11: D, Diode_SMD:D_0201_0603Metric, F.Cu at (153.6, 128.6)
- added D2: NeoPixel_THT, LED_SMD:LED_WS2812_PLCC6_5.0x5.0mm_P1.6mm, F.Cu at (125.5, 67.5)
- added D3: NeoPixel_THT, LED_SMD:LED_WS2812_PLCC6_5.0x5.0mm_P1.6mm, F.Cu at (113.5, 73.6)
- added D4: NeoPixel_THT, LED_SMD:LED_WS2812_PLCC6_5.0x5.0mm_P1.6mm, F.Cu at (106.0, 83.1)
- added D5: NeoPixel_THT, LED_SMD:LED_WS2812_PLCC6_5.0x5.0mm_P1.6mm, F.Cu at (101.5, 93.6)
- added D6: NeoPixel_THT, LED_SMD:LED_WS2812_PLCC6_5.0x5.0mm_P1.6mm, F.Cu at (99.5, 103.5)
- added D7: NeoPixel_THT, LED_SMD:LED_WS2812_PLCC6_5.0x5.0mm_P1.6mm, F.Cu at (100.0, 114.0)
- added D8: NeoPixel_THT, LED_SMD:LED_WS2812_PLCC6_5.0x5.0mm_P1.6mm, F.Cu at (104.0, 124.1)
- added D9: C35722, Diode_SMD:D_0201_0603Metric, F.Cu at (153.6, 125.1)
- added J2: USB_C_Receptacle_USB2.0_16P, Connector_USB:USB_C_Receptacle_Amphenol_12401548E4-2A, F.Cu at (166.9, 107.6)
- added R2: 5k1, Resistor_SMD:R_0805_2012Metric_Pad1.20x1.40mm_HandSolder, F.Cu at (149.8, 125.7)
- added R3: 5k1, Resistor_SMD:R_0805_2012Metric_Pad1.20x1.40mm_HandSolder, F.Cu at (149.8, 128.7)
- added R4: 1k, Resistor_SMD:R_0805_2012Metric_Pad1.20x1.40mm_HandSolder, F.Cu at (149.8, 131.6)
- added R5: 1k, Resistor_SMD:R_0805_2012Metric_Pad1.20x1.40mm_HandSolder, F.Cu at (149.8, 134.6)
- added R6: 10k, Resistor_SMD:R_0805_2012Metric_Pad1.20x1.40mm_HandSolder, F.Cu at (149.8, 137.5)
- added U2: ADXL343, Package_LGA:LGA-14_3x5mm_P0.8mm_LayoutBorder1x6y, F.Cu at (131.5, 140.4)
- added U3: CH340N, Package_SO:SOP-8_3.9x4.9mm_P1.27mm, F.Cu at (151.6, 142.4)
Connections:
- R1 pad 2: Net-(SW1-B) -> VCC
- SW1 pad 2: Net-(SW1-B) -> VCC
- U1 pad 29: Net-(SW1-B) -> VCC
Routing:
- net GND: track 116.9 -> 240.9 mm, vias 7 -> 9
- net Net-(J2-CC2): track 0.00 -> 58.2 mm
- net /UD-: track 0.00 -> 45.7 mm
- net /UD+: track 0.00 -> 44.6 mm, vias 0 -> 1
- net A4: track 0.00 -> 40.8 mm, vias 0 -> 2
- net A5: track 0.00 -> 40.6 mm, vias 0 -> 2
- net VCC: track 105.1 -> 144.3 mm, vias 0 -> 2
- net Net-(SW1-B): track 39.2 -> 0.00 mm, vias 2 -> 0
- net D7: track 0.00 -> 39.0 mm
- net /RESET: track 0.00 -> 38.6 mm, vias 0 -> 2
- net D6: track 0.00 -> 38.1 mm
- net D5: track 0.00 -> 37.6 mm
- net D2: track 0.00 -> 36.6 mm, vias 0 -> 2
- net VBUS: track 0.00 -> 35.7 mm, vias 0 -> 2
- net D4: track 0.00 -> 34.7 mm, vias 0 -> 1
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
Commit message: 3 hr
Added barometer / altimeter, battery, arduino pinout
Parts:
- added A1: Arduino_Nano_v3.x, Module:Arduino_Nano_WithMountingHoles, F.Cu at (146.9, 81.0)
- added C10: 100 nF, Capacitor_SMD:C_0805_2012Metric_Pad1.18x1.45mm_HandSolder, F.Cu at (43.6, 54.8)
- added C11: 1 uF, Capacitor_SMD:C_0805_2012Metric_Pad1.18x1.45mm_HandSolder, F.Cu at (43.6, 57.8)
- added D12: LED, Diode_SMD:D_1206_3216Metric_Pad1.42x1.75mm_HandSolder, F.Cu at (58.5, 46.0)
- added D13: LED, Diode_SMD:D_1206_3216Metric_Pad1.42x1.75mm_HandSolder, F.Cu at (58.5, 49.4)
- added D14: RED, Diode_SMD:D_1206_3216Metric_Pad1.42x1.75mm_HandSolder, F.Cu at (58.5, 52.8)
- added D15: GREEN, Diode_SMD:D_1206_3216Metric_Pad1.42x1.75mm_HandSolder, F.Cu at (58.5, 56.1)
- added D16: C8678, Diode_SMD:D_1206_3216Metric, F.Cu at (86.6, 72.5)
- added Q1: AO3401A, Package_TO_SOT_SMD:SOT-23, F.Cu at (38.8, 64.7)
- added R10: 10k, Resistor_SMD:R_0805_2012Metric_Pad1.20x1.40mm_HandSolder, F.Cu at (53.1, 54.6)
- added R7: 1k5, Resistor_SMD:R_0805_2012Metric_Pad1.20x1.40mm_HandSolder, F.Cu at (174.0, 58.0)
- added R8: 4k7, Resistor_SMD:R_0805_2012Metric_Pad1.20x1.40mm_HandSolder, F.Cu at (53.1, 48.7)
- added R9: 1k, Resistor_SMD:R_0805_2012Metric_Pad1.20x1.40mm_HandSolder, F.Cu at (53.1, 51.6)
- added U4: MPL3115A2, Package_LGA:NXP_LGA-8_3x5mm_P1.25mm_H1.1mm, F.Cu at (72.3, 81.4)
- added U5: TP4057, Package_TO_SOT_SMD:TSOT-23-5, F.Cu at (175.4, 53.0)
- added U6: XC6206PxxxMR, Package_TO_SOT_SMD:SOT-23-3, F.Cu at (91.4, 83.5)
- C5: value 100 nF -> 1 uF
- C7: value C -> 100 nF
- D10: value D -> YELLOW; footprint Diode_SMD:D_0201_0603Metric -> Diode_SMD:D_SMC_Handsoldering
- D11: value D -> GREEN; footprint Diode_SMD:D_0201_0603Metric -> Diode_SMD:D_SMC_Handsoldering
- D9: value C35722 -> C8678; footprint Diode_SMD:D_0201_0603Metric -> Diode_SMD:D_SMC_Handsoldering
- R4, R5: value 1k -> 330R
- moved D9 144.1 mm to (60.7, 15.1)
- moved D10 139.5 mm to (60.7, 22.8)
- moved C7 133.0 mm to (43.6, 45.8)
- moved R4 127.3 mm to (48.4, 54.6)
- moved R5 127.3 mm to (48.4, 57.5)
- moved C9 126.7 mm to (43.6, 51.8), turned to 0 degrees
- moved C5 126.1 mm to (38.8, 57.8)
- moved C8 124.6 mm to (43.6, 48.8), turned to 0 degrees
- moved C6 123.4 mm to (36.5, 70.0), turned to 90 degrees
- moved SW1 119.4 mm to (28.0, 69.9)
- moved D8 111.0 mm to (49.0, 27.7)
- moved J1 110.2 mm to (55.5, 36.8)
- moved D1 109.7 mm to (40.6, 14.5)
- moved R1 106.9 mm to (48.4, 45.8)
- moved D7 106.0 mm to (49.0, 21.1)
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Connections:
- C5 pad 1: GND -> Vdrive
- C5 pad 2: Net-(U3-V3) -> GND
- C6 pad 1: Net-(U3-VCC) -> VCC
- D9 pad 1: VCC -> VBUS
- D9 pad 2: VBUS -> /USB_P
- J2 pad A4: VBUS -> /USB_P
- J2 pad A9: VBUS -> /USB_P
- J2 pad B4: VBUS -> /USB_P
- J2 pad B9: VBUS -> /USB_P
- R4 pad 1: Net-(U3-VCC) -> VCC
- R5 pad 1: Net-(U3-VCC) -> VCC
- U3 pad 5: Net-(U3-VCC) -> VCC
- U3 pad 8: Net-(U3-V3) -> VCC
Routing:
- net GND: track 240.9 -> 71.7 mm, vias 9 -> 2
- net VCC: track 144.3 -> 74.6 mm, vias 2 -> 0
- net /UD-: track 45.7 -> 0.00 mm
- net Net-(J2-CC2): track 58.2 -> 12.8 mm
- net /UD+: track 44.6 -> 0.00 mm, vias 1 -> 0
- net D7: track 39.0 -> 0.00 mm
- net /RESET: track 38.6 -> 0.00 mm, vias 2 -> 0
- net D6: track 38.1 -> 0.00 mm
- net D5: track 37.6 -> 0.00 mm
- net D2: track 36.6 -> 0.00 mm, vias 2 -> 0
- net VBUS: track 35.7 -> 0.00 mm, vias 2 -> 0
- net D4: track 34.7 -> 0.00 mm, vias 1 -> 0
- net D3: track 34.2 -> 0.00 mm, vias 2 -> 0
- net A4: track 40.8 -> 9.96 mm, vias 2 -> 0
- net D12: track 30.0 -> 0.00 mm, vias 2 -> 0
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Other:
- board size 91.1 x 91.1 mm -> 219.5 x 123 mm

Commit message: Another hour
Finished up the schematic (at least I hope) & started working (~ 1/2 way done), with the actual PCB layout.
Parts:
- added R11: 4.7k, Resistor_SMD:R_0805_2012Metric_Pad1.20x1.40mm_HandSolder, F.Cu at (170.5, 114.5)
- added R12: 4.7k, Resistor_SMD:R_0805_2012Metric_Pad1.20x1.40mm_HandSolder, F.Cu at (170.0, 110.0)
- added R13: 1k, Resistor_SMD:R_0805_2012Metric_Pad1.20x1.40mm_HandSolder, F.Cu at (147.7, 103.5)
- added R14: 1k, Resistor_SMD:R_0805_2012Metric_Pad1.20x1.40mm_HandSolder, F.Cu at (151.9, 98.8)
- D16: footprint Diode_SMD:D_1206_3216Metric -> Diode_SMD:D_SMA
- moved J1 157.4 mm to (181.3, 131.4), turned to 180 degrees
- moved C8 149.8 mm to (177.0, 117.0)
- moved C9 144.9 mm to (173.5, 116.0)
- moved C6 119.1 mm to (153.6, 48.4), turned to 180 degrees
- moved R4 115.1 mm to (162.6, 39.9), turned to -90 degrees
- moved C5 114.9 mm to (149.9, 86.8), turned to 180 degrees
- moved C11 112.0 mm to (150.7, 90.3), turned to 90 degrees
- moved C10 111.7 mm to (154.4, 41.3), turned to -90 degrees
- moved Q1 110.1 mm to (148.9, 62.7), turned to -90 degrees
- moved C7 109.3 mm to (148.7, 75.8), turned to -90 degrees
- moved R6 106.6 mm to (179.5, 109.0), turned to 0 degrees
- moved SW1 104.5 mm to (117.3, 124.0), turned to 90 degrees
- moved R10 103.8 mm to (154.9, 74.7)
- moved R5 101.1 mm to (147.1, 35.6), turned to 90 degrees
- moved R1 100.7 mm to (120.8, 115.7)
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Connections:
- D1 pad 4: unconnected-(D1-DIN-Pad4) -> D8
- D2 pad 4: unconnected-(D2-DIN-Pad4) -> D1
Routing:
- net VCC: track 74.6 -> 259.0 mm, vias 0 -> 2
- net D0: track 0.00 -> 163.3 mm, vias 0 -> 4
- net VBUS: track 0.00 -> 139.7 mm, vias 0 -> 6
- net /RESET: track 0.00 -> 119.1 mm
- net A5: track 14.7 -> 89.6 mm
- net D1: track 0.00 -> 58.9 mm, vias 0 -> 2
- net A4: track 9.96 -> 67.7 mm, vias 0 -> 2
- net Net-(D11-A): track 0.00 -> 49.5 mm, vias 0 -> 2
- net /UD-: track 0.00 -> 42.2 mm
- net A6: track 0.00 -> 39.7 mm
- net D11: track 0.00 -> 38.3 mm
- net Vdrive: track 0.00 -> 38.2 mm, vias 0 -> 2
- net D13: track 0.00 -> 35.1 mm, vias 0 -> 1
- net Net-(U3-~{RTS}): track 0.00 -> 34.9 mm
- net /UD+: track 0.00 -> 31.6 mm, vias 0 -> 2
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Other:
- board size 219.5 x 123 mm -> 244.5 x 187.3 mm

Commit message: Almost done
Basically just need to convert everything to JLCPCB components now, and then I should be good to go.
Parts:
- removed U4: MPL3115A2, Package_LGA:NXP_LGA-8_3x5mm_P1.25mm_H1.1mm
- added U7: MS5607-02BA, Package_LGA:LGA-8_3x5mm_P1.25mm, F.Cu at (113.0, 135.0)
- moved D7 173.4 mm to (177.6, 180.9)
- moved D6 171.4 mm to (165.0, 181.0)
- moved D8 167.5 mm to (164.5, 189.9)
- moved D4 163.2 mm to (180.1, 170.4)
- moved D3 160.2 mm to (169.5, 169.9)
- moved D2 158.2 mm to (158.5, 169.9), turned to 180 degrees
- moved D1 157.5 mm to (148.0, 170.0), turned to 180 degrees
- moved D5 149.1 mm to (155.1, 181.0)
- moved R7 111.4 mm to (71.0, 133.0), turned to 90 degrees
- moved U5 99.4 mm to (77.5, 134.6), turned to 90 degrees
- moved D11 99.1 mm to (122.5, 117.5), turned to 180 degrees
- moved C4 97.4 mm to (139.5, 134.5), turned to 180 degrees
- moved R4 94.8 mm to (101.0, 112.0), turned to 180 degrees
- moved C3 92.3 mm to (139.5, 122.0)
- moved D12 92.2 mm to (93.7, 128.0), turned to 90 degrees
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Routing:
- net A4: track 67.7 -> 241.7 mm, vias 2 -> 9
- net VCC: track 259.0 -> 386.3 mm, vias 2 -> 14
- net D3: track 7.86 -> 122.6 mm, vias 0 -> 4
- net D1: track 58.9 -> 172.4 mm, vias 2 -> 10
- net D4: track 7.14 -> 111.9 mm, vias 0 -> 1
- net D7: track 4.73 -> 99.3 mm, vias 0 -> 1
- net VBUS: track 139.7 -> 231.9 mm, vias 6 -> 19
- net D12: track 29.9 -> 120.7 mm
- net A5: track 89.6 -> 175.0 mm, vias 2 -> 8
- net D6: track 4.44 -> 89.1 mm, vias 0 -> 7
- net D11: track 38.3 -> 111.5 mm, vias 0 -> 4
- net D5: track 4.28 -> 66.8 mm, vias 0 -> 2
- net /RESET: track 119.1 -> 62.7 mm, vias 0 -> 1
- net D2: track 25.4 -> 77.6 mm, vias 0 -> 1
- net A3: track 4.80 -> 56.7 mm, vias 0 -> 2
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Other:
- board size 244.5 x 187.3 mm -> 407.5 x 312.2 mm

Commit message: FINISHED
Final assignments, and shrinked board.
Other:
- board size 407.5 x 312.2 mm -> 298.3 x 219.1 mm
Changed lines of the file:
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@@
 	(gr_poly
 		(pts
-			(xy 164.909354 -67.183566) (xy 165.570785 -46.016897) (xy 166.893722 -34.772095) (xy 172.185375 -48.662715)
-			(xy 225.763484 -39.402289) (xy 229.070789 -37.417912) (xy 229.732238 -28.818964) (xy 229.732238 -20.881457)
-			(xy 229.070789 -10.959582) (xy 225.763484 -8.313736) (xy 170.862456 -1.037707) (xy 184.753066 105.457063)
-			(xy 256.190559 105.457063) (xy 367.315551 120.67061) (xy 367.315551 154.404989) (xy 365.331184 159.696622)
-			(xy 361.362449 162.342477) (xy 258.174964 166.972681) (xy 184.753066 166.972681) (xy 184.091617 189.462247)
-			(xy 180.784331 215.259137) (xy 179.461413 219.889341) (xy 177.477046 222.535177) (xy 173.508292 223.858076)
-			(xy 168.878089 223.858076) (xy 168.21664 227.16538) (xy 201.950999 227.826848) (xy 201.950999 229.149747)
-			(xy 167.555171 229.149747) (xy 166.232234 234.441457) (xy 163.586398 239.071622) (xy 160.940581 234.441457)
-			(xy 159.617664 229.149747) (xy 124.560367 229.149747) (xy 124.560367 227.826848) (xy 158.956214 227.16538)
-			(xy 158.294746 223.858076) (xy 153.664543 223.858076) (xy 149.695789 222.535177) (xy 147.711421 219.889341)
-			(xy 146.388484 215.259137) (xy 143.081199 189.462247) (xy 142.41973 166.972681) (xy 68.997861 166.972681)
-			(xy -34.189632 161.681028) (xy -38.158383 159.696661) (xy -40.142757 154.404989) (xy -40.142757 120.670629)
-			(xy 70.982238 105.457063) (xy 142.41973 105.457063) (xy 156.310359 -1.037707) (xy 101.409331 -8.313736)
-			(xy 98.102037 -10.959582) (xy 97.440578 -20.881457) (xy 97.440578 -28.818964) (xy 98.102037 -37.417912)
-			(xy 101.409331 -39.402289) (xy 154.98746 -48.662715) (xy 160.279113 -34.772095) (xy 161.60205 -46.016897)
-			(xy 162.263499 -67.183566) (xy 163.586417 -73.136701)
+			(xy 186.236984 102.929542) (xy 257.674476 102.929542) (xy 259.658844 164.44516) (xy 186.236984 164.44516)
+			(xy 185.575516 186.934726) (xy 182.26823 212.731617) (xy 180.945332 217.36182) (xy 178.960926 220.007656)
+			(xy 174.992191 221.330555) (xy 170.361969 221.330555) (xy 169.700539 224.637859) (xy 169.039051 226.622226)
+			(xy 167.716152 231.913936) (xy 165.070316 236.544101) (xy 162.42448 231.913936) (xy 161.101563 226.622226)
+			(xy 160.440094 224.637859) (xy 159.778664 221.330555) (xy 155.148441 221.330555) (xy 151.179688 220.007656)
+			(xy 149.19532 217.36182) (xy 147.872402 212.731617) (xy 144.565098 186.934726) (xy 143.903648 164.44516)
+			(xy 70.481779 164.44516) (xy -32.70572 159.153507) (xy -36.674469 157.169101) (xy -38.658844 151.877449)
+			(xy -38.658844 118.143089) (xy 72.466156 102.929542) (xy 143.903648 102.929542) (xy 124.820587 18.891256)
+			(xy 214.395267 17.4559)
 		)
 		(stroke
@@
 	)
 	(group ""
-		(members "c448960c-46f3-4793-baa3-0003805b6012")
+		(members "d02a1e8e-4ca2-450c-ab32-7de521040f77")
 	)
 )
