File: src/name.kicad_pcb (KiCad board)
At the start: 2 copper layers, 298.3 x 219.1 mm, 53 parts, among them J1 Conn_02x03_Odd_Even, J2 USB_C_Receptacle_USB2.0_16P, Q1 AO3401A, SW1 SW_SPST, U1 ATmega328P-A, U2 ADXL343, U3 CH340N, U5 TP4057, U6 XC6206PxxxMR, U7 MS5607-02BA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

Commit message: 1/2 hr
Spent a lot of time fiddling with JLCPCB, before deciding to use OSHPark
Other:
- board size 298.3 x 219.1 mm -> 148.5 x 217.7 mm
Changed lines of the file:
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@@
 		(tags "USB C Type-C Receptacle Hybrid")
 		(property "Reference" "J2"
-			(at 0 -6.36 360)
+			(at 0 -6.36 0)
 			(layer "F.SilkS")
 			(effects
@@
 		)
 		(property "Value" "USB_C_Receptacle_USB2.0_16P"
-			(at 0 6.14 360)
+			(at 0 6.14 0)
 			(layer "F.Fab")
 			(hide yes)
@@
 		)
 		(fp_text user "${REFERENCE}"
-			(at 0 0 360)
+			(at 0 0 0)
 			(layer "F.Fab")
 			(effects
@@
 		(tags "Diode SMC (DO-214AB) Handsoldering")
 		(property "Reference" "D11"
-			(at 0 -4.1 360)
+			(at 0 -4.1 0)
 			(layer "F.SilkS")
 			(effects
@@
 		)
 		(property "Value" "GREEN"
-			(at 0 4.2 360)
+			(at 0 4.2 0)
 			(layer "F.Fab")
 			(effects
@@
 		)
 		(fp_text user "${REFERENCE}"
-			(at 0 -1.5 360)
+			(at 0 -1.5 0)
 			(layer "F.Fab")
 			(effects
@@
 		(tags "LED RGB NeoPixel")
 		(property "Reference" "D2"
-			(at 0 -3.5 360)
+			(at 0 -3.5 0)
 			(layer "F.SilkS")
 			(effects
@@
 		)
 		(property "Value" "NeoPixel_THT"
-			(at 0 4 360)
+			(at 0 4 0)
 			(layer "F.Fab")
 			(effects
@@
 		)
 		(fp_text user "${REFERENCE}"
-			(at 0 0 360)
+			(at 0 0 0)
 			(layer "F.Fab")
 			(effects
@@
 		(tags "capacitor handsolder")
 		(property "Reference" "C4"
-			(at 0 -1.68 360)
+			(at 0 -1.68 0)
 			(layer "F.SilkS")
 			(effects
@@
 		)
 		(property "Value" "12pF"
-			(at 0 1.68 360)
+			(at 0 1.68 0)
 			(layer "F.Fab")
 			(effects
@@
 		)
 		(fp_text user "${REFERENCE}"
-			(at 0 0 360)
+			(at 0 0 0)
 			(layer "F.Fab")
 			(effects
@@
 		(tags "LED RGB NeoPixel")
 		(property "Reference" "D1"
-			(at 0 -3.5 360)
+			(at 0 -3.5 0)
 			(layer "F.SilkS")
 			(effects
@@
 		)
 		(property "Value" "NeoPixel_THT"
-			(at 0 4 360)
+			(at 0 4 0)
 			(layer "F.Fab")
 			(effects
@@
 		)
 		(fp_text user "${REFERENCE}"
-			(at 0 0 360)
+			(at 0 0 0)
 			(layer "F.Fab")
 			(effects
@@
 		)
 		(fp_text user "${REFERENCE}"
-			(at 0 0 360)
+			(at 0 0 0)
 			(layer "F.Fab")
 			(effects
@@
 		(tags "capacitor handsolder")
 		(property "Reference" "C11"
-			(at 0 -1.68 360)
+			(at 0 -1.68 0)
 			(layer "F.SilkS")
 			(effects
@@
 		)
 		(property "Value" "1 uF"
-			(at 0 1.68 360)
+			(at 0 1.68 0)
 			(layer "F.Fab")
 			(effects
@@
 		)
 		(fp_text user "${REFERENCE}"
-			(at 0 0 360)
+			(at 0 0 0)
 			(layer "F.Fab")
 			(effects
@@
 		(tags "resistor handsolder")
 		(property "Reference" "R9"
-			(at 0 -1.65 360)
+			(at 0 -1.65 0)
 			(layer "F.SilkS")
 			(effects
@@
 		)
 		(property "Value" "1k"
-			(at 0 1.65 360)
+			(at 0 1.65 0)
 			(layer "F.Fab")
 			(effects
@@
 		)
 		(fp_text user "${REFERENCE}"
-			(at 0 0 360)
+			(at 0 0 0)
 			(layer "F.Fab")
 			(effects
@@
 		(tags "Through hole pin header THT 2x03 2.54mm double row")
 		(property "Reference" "J1"
-			(at 1.27 -2.33 360)
+			(at 1.27 -2.33 0)
 			(layer "F.SilkS")
 			(effects
@@
 		)
 		(property "Value" "Conn_02x03_Odd_Even"
-			(at 1.27 7.41 360)
+			(at 1.27 7.41 0)
 			(layer "F.Fab")
 			(effects
@@
 		(tags "diode handsolder")
 		(property "Reference" "D14"
-			(at 0 -1.82 360)
+			(at 0 -1.82 0)
 			(layer "F.SilkS")
 			(effects
@@
 		)
 		(property "Value" "RED"
-			(at 0 1.82 360)
+			(at 0 1.82 0)
 			(layer "F.Fab")
 			(effects
@@
 		)
 		(fp_text user "${REFERENCE}"
-			(at 0 0 360)
+			(at 0 0 0)
 			(layer "F.Fab")
 			(effects
@@
 		(tags "resistor handsolder")
 		(property "Reference" "R4"
-			(at 0 -1.65 360)
+			(at 0 -1.65 0)
 			(layer "F.SilkS")
 			(effects
@@
 		)
 		(property "Value" "330R"
-			(at 0 1.65 360)
+			(at 0 1.65 0)
 			(layer "F.Fab")
 			(effects
@@
 		)
 		(fp_text user "${REFERENCE}"
-			(at 0 0 360)
+			(at 0 0 0)
 			(layer "F.Fab")
 			(effects
@@
 		(tags "capacitor handsolder")
 		(property "Reference" "C6"
-			(at 0 -1.68 360)
+			(at 0 -1.68 0)
 			(layer "F.SilkS")
 			(effects
@@
 		)
 		(property "Value" "100 nF"
-			(at 0 1.68 360)
+			(at 0 1.68 0)
 			(layer "F.Fab")
 			(effects
@@
 		)
 		(fp_text user "${REFERENCE}"
-			(at 0 0 360)
+			(at 0 0 0)
 			(layer "F.Fab")
 			(effects
@@
 	(gr_poly
 		(pts
-			(xy 186.236984 102.929542) (xy 257.674476 102.929542) (xy 259.658844 164.44516) (xy 186.236984 164.44516)
-			(xy 185.575516 186.934726) (xy 182.26823 212.731617) (xy 180.945332 217.36182) (xy 178.960926 220.007656)
-			(xy 174.992191 221.330555) (xy 170.361969 221.330555) (xy 169.700539 224.637859) (xy 169.039051 226.622226)
-			(xy 167.716152 231.913936) (xy 165.070316 236.544101) (xy 162.42448 231.913936) (xy 161.101563 226.622226)
-			(xy 160.440094 224.637859) (xy 159.778664 221.330555) (xy 155.148441 221.330555) (xy 151.179688 220.007656)
-			(xy 149.19532 217.36182) (xy 147.872402 212.731617) (xy 144.565098 186.934726) (xy 143.903648 164.44516)
-			(xy 70.481779 164.44516) (xy -32.70572 159.153507) (xy -36.674469 157.169101) (xy -38.658844 151.877449)
-			(xy -38.658844 118.143089) (xy 72.466156 102.929542) (xy 143.903648 102.929542) (xy 124.820587 18.891256)
-			(xy 214.395267 17.4559)
+			(xy 194.5 74) (xy 208 137.5) (xy 185.575516 190.434726) (xy 182.26823 212.731617) (xy 180.945332 217.36182)
+			(xy 178.960926 220.007656) (xy 174.992191 221.330555) (xy 170.361969 221.330555) (xy 169.700539 224.637859)
+			(xy 169.039051 226.622226) (xy 167.716152 231.913936) (xy 165.070316 236.544101) (xy 162.42448 231.913936)
+			(xy 161.101563 226.622226) (xy 160.440094 224.637859) (xy 159.778664 221.330555) (xy 155.148441 221.330555)
+			(xy 151.179688 220.007656) (xy 149.19532 217.36182) (xy 147.872402 212.731617) (xy 144.565098 186.934726)
+			(xy 143.903648 164.44516) (xy 74.481779 163.44516) (xy 59.466156 102.429542) (xy 143.903648 102.929542)
+			(xy 124.820587 18.891256) (xy 195.895267 18.9559)
 		)
 		(stroke
